File: hardware/buck-boost.kicad_pcb (KiCad board)
At the start: 2 copper layers, 67.5 x 67.5 mm, 67 parts, among them J1 FC681465, J2 301-021-12, J3 301-021-12, J4 DS1013-20S, J5 PLS-2, Y1 HC49-S

Commit message: change reverse polarity protection from low side to high side
1. polarity protection schematic changes
2. new tracing for analog gnd part of pcb (gnda still not in shematic)
Parts:
- VT3: value IRLML0030TRPBF -> IRLML9301TRPbF
- moved C25 5.60 mm to (144.2, 116.8), turned to 180 degrees
- moved C13 4.86 mm to (124.8, 109.5), turned to 90 degrees
- moved R5 4.70 mm to (140.0, 70.8), turned to 270 degrees
- moved VD1 3.16 mm to (141.8, 67.2), turned to 180 degrees
- moved VT3 1.58 mm to (143.0, 70.2), turned to 90 degrees
- moved D7 1.50 mm to (124.0, 113.2)
- moved C24 1.25 mm to (135.0, 119.5)
- moved R11 1.25 mm to (121.2, 115.5)
- moved C20 0.61 mm to (145.4, 115.4)
- moved C12 0.25 mm to (126.2, 109.5)
Connections:
- J1 pad 1: /Vin -> Net-(J1-Pad1)
- J1 pad 2: Net-(J1-Pad2) -> GND
- J1 pad 3: Net-(J1-Pad2) -> GND
- J3 pad 1: /Vin -> Net-(J1-Pad1)
- J3 pad 2: Net-(J1-Pad2) -> GND
- R5 pad 1: /Vin -> Net-(R5-Pad1)
- R5 pad 2: Net-(R5-Pad2) -> GND
- VD1 pad 1: Net-(R5-Pad2) -> Net-(J1-Pad1)
- VD1 pad 2: GND -> Net-(R5-Pad1)
- VT3 pad 1: Net-(R5-Pad2) -> Net-(R5-Pad1)
- VT3 pad 2: GND -> /Vin
- VT3 pad 3: Net-(J1-Pad2) -> Net-(J1-Pad1)
Routing:
- net GND: track 147.3 -> 160.7 mm, vias 30 -> 23
- net Net-(R5-Pad1): track 0.00 -> 5.01 mm
- net Net-(R5-Pad2): track 3.88 -> 0.00 mm
- net +3V3: track 25.0 -> 28.8 mm, vias 0 -> 2
- net Net-(C12-Pad1): track 17.4 -> 21.0 mm
- added copper zone on F.Cu, net Net-(J1-Pad1)
- removed copper zone on F.Cu, net Net-(J1-Pad2)
